File: Hardware/Testbench_stepper/connectors.kicad_sch (KiCad schematic)
At the start: 2 parts, among them CN11 Conn_02x35_Odd_Even, CN12 Conn_02x35_Odd_Even

Commit message: hw: schematic update
Parts:
- added J?: Conn_01x08_Female, Connector_PinHeader_2.54mm:PinHeader_1x08_P2.54mm_Vertical, symbol Connector:Conn_01x08_Female
- added J?: Conn_01x02_Female, Connector_PinHeader_2.54mm:PinHeader_1x02_P2.54mm_Vertical, symbol Connector:Conn_01x02_Female
Connections:
- new net +12V: J?.1 (Pin_1), J?.2 (Pin_2)
- new net +2V5: J?.7 (Pin_7), J?.8 (Pin_8)
- new net GND: J?.5 (Pin_5), J?.6 (Pin_6)
- new net TRQ: J?.3 (Pin_3), J?.4 (Pin_4)
- new net V_SUPPLY+: J?.1 (Pin_1)
- new net V_SUPPLY-: J?.2 (Pin_2)
- no-connect marks 0 -> 140
Other:
- note added: "BLACK"
- note added: "BROWN"
- note added: "GREY"
- note added: "TORQUE SENSOR CONNECTOR"
- note added: "The output Vref is a constant 2.5 V output and represents the virtual zero point for direct +/-torque measurement."
- note added: "V_SUPPLY"
- note added: "WHITE"
