File: Hardware/Testbench_stepper/sensing.kicad_sch (KiCad schematic)
At the start: 1 part, among them U2 LEM-CAS-6-NP

Commit message: hw: schematic update
Parts:
- added C? (x3): 100n, symbol Device:C
- added C? (x3): 0.1u, symbol Device:C
- added R? (x3): 10k, symbol Device:R
- added R?: 33K, symbol Device:R
- added R?: 6k2, symbol Device:R
- added R?: 6K2, symbol Device:R
- added R? (x2): 3k3, symbol Device:R
- added R?: 3K3, symbol Device:R
- added U? (x3): LM358P, Package_TO_SOT_SMD:SOT-23-8, symbol EncoderLib:LM358P
Connections:
- net +5V: now reaches U2.1 (VDD)
- net +5V: now also C?.1, C?.1, U?.8 (V+), U?.8 (V+)
- net GND: now reaches U2.2 (GND)
- net GND: now also C?.2, C?.2, C?.2, C?.2, C?.2, C?.2, R?.2, R?.2, R?.2, U?.4 (V-), U?.4 (V-), U?.4 (V-)
- net CURRENT_SENSOR_OUTPUT: now reaches U2.3 (Out)
- net CURRENT_SENSOR_OUTPUT: now also U?.3 (IN1+)
- net COIL_IN: now reaches U2.4 (IN_COIL_1)
- net COIL_IN: now also U2.5 (IN_COIL_2), U2.6 (IN_COIL_3)
- net COIL_OUT: now reaches U2.7 (OUT_COIL_1)
- net COIL_OUT: now also U2.8 (OUT_COIL_2), U2.9 (OUT_COIL_3)
- new net: C?.1, R?.1, R?.1 (x3)
- new net ADC_BUFF_CURRENT: U?.6 (IN2-), U?.7 (OUT2)
- new net ADC_BUFF_TRQ: U?.6 (IN2-), U?.7 (OUT2)
- new net ADC_BUFF_V_SUPPLY: U?.6 (IN2-), U?.7 (OUT2)
- new net ADC_CURRENT: R?.1, R?.2, U?.5 (IN2+)
- new net ADC_TRQ: R?.1, R?.2, U?.5 (IN2+)
- new net ADC_V_SUPPLY: R?.1, R?.2, U?.5 (IN2+)
- new net CURRENT_BUFF: R?.2, U?.1 (OUT1), U?.2 (IN1-)
- new net TRQ: U?.3 (IN1+)
- new net TRQ_BUFF: R?.2, U?.1 (OUT1), U?.2 (IN1-)
- new net V_SUPPLY: C?.1, U?.3 (IN1+), U?.8 (V+)
- new net V_SUPPLY_BUFF: R?.2, U?.1 (OUT1), U?.2 (IN1-)
Other:
- note added: "Dual Op-Amp"
- note added: "Is it correct sot23-8 as package?"
- note added: "prev was 12v"
- note added: "prev was: up: 2k down: 33k"
- moved on the sheet: U2
