File: Hardware/Testbench_stepper/testbench_stepper.kicad_pcb (KiCad board)
At the start: 2 copper layers, 74.3 x 120.1 mm, 3 parts, among them CN11 Conn_02x35_Odd_Even, CN12 Conn_02x35_Odd_Even, U2 LEM-CAS-6-NP

Commit message: hw: schematic update
Parts:
- added J1: Conn_01x08_Male, Connector_PinHeader_2.54mm:PinHeader_1x08_P2.54mm_Vertical, F.Cu at (157.5, 34.0)
Changed lines of the file:
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@@
   (net 148 "unconnected-(U2-Pad8)")
   (net 149 "unconnected-(U2-Pad9)")
+  (net 150 "/Connectors/VDD")
+  (net 151 "/Connectors/TRQ")
+  (net 152 "/Connectors/GND")
+  (net 153 "/Connectors/VREF")
   (footprint "Sensing lib:LEM-CAS-6-NP" (layer "F.Cu")
     (at 140.716 29.718)
@@
       (offset (xyz 0 0 0))
       (scale (xyz 1 1 1))
+      (rotate (xyz 0 0 0))
+    )
+  )
+  (footprint "Connector_PinHeader_2.54mm:PinHeader_1x08_P2.54mm_Vertical" (layer "F.Cu")
+    (at 157.48 34.036 90)
+    (descr "Through hole straight pin header, 1x08, 2.54mm pitch, single row")
+    (tags "Through hole pin header THT 1x08 2.54mm single row")
+    (property "Sheetfile" "connectors.kicad_sch")
+    (property "Sheetname" "Connectors")
+    (attr through_hole)
+    (fp_text reference "J1" (at 0 -2.33 90) (layer "F.SilkS")
+      (effects (font (size 1 1) (thickness 0.15)))
+    )
+    (fp_text value "Conn_01x08_Male" (at 0 20.11 90) (layer "F.Fab")
+      (effects (font (size 1 1) (thickness 0.15)))
+    )
+    (fp_text user "${REFERENCE}" (at 0 8.89) (layer "F.Fab")
+      (effects (font (size 1 1) (thickness 0.15)))
+    )
+    (fp_line (start -1.33 19.11) (end 1.33 19.11) (layer "F.SilkS") (width 0.12))
+    (fp_line (start -1.33 0) (end -1.33 -1.33) (layer "F.SilkS") (width 0.12))
+    (fp_line (start -1.33 1.27) (end 1.33 1.27) (layer "F.SilkS") (width 0.12))
+    (fp_line (start 1.33 1.27) (end 1.33 19.11) (layer "F.SilkS") (width 0.12))
+    (fp_line (start -1.33 -1.33) (end 0 -1.33) (layer "F.SilkS") (width 0.12))
+    (fp_line (start -1.33 1.27) (end -1.33 19.11) (layer "F.SilkS") (width 0.12))
+    (fp_line (start 1.8 -1.8) (end -1.8 -1.8) (layer "F.CrtYd") (width 0.05))
+    (fp_line (start -1.8 -1.8) (end -1.8 19.55) (layer "F.CrtYd") (width 0.05))
+    (fp_line (start 1.8 19.55) (end 1.8 -1.8) (layer "F.CrtYd") (width 0.05))
+    (fp_line (start -1.8 19.55) (end 1.8 19.55) (layer "F.CrtYd") (width 0.05))
+    (fp_line (start -0.635 -1.27) (end 1.27 -1.27) (layer "F.Fab") (width 0.1))
+    (fp_line (start 1.27 19.05) (end -1.27 19.05) (layer "F.Fab") (width 0.1))
+    (fp_line (start -1.27 -0.635) (end -0.635 -1.27) (layer "F.Fab") (width 0.1))
+    (fp_line (start -1.27 19.05) (end -1.27 -0.635) (layer "F.Fab") (width 0.1))
+    (fp_line (start 1.27 -1.27) (end 1.27 19.05) (layer "F.Fab") (width 0.1))
+    (pad "1" thru_hole rect (at 0 0 90) (size 1.7 1.7) (drill 1) (layers *.Cu *.Mask)
+      (net 150 "/Connectors/VDD") (pinfunction "Pin_1") (pintype "passive"))
+    (pad "2" thru_hole oval (at 0 2.54 90) (size 1.7 1.7) (drill 1) (layers *.Cu *.Mask)
+      (net 150 "/Connectors/VDD") (pinfunction "Pin_2") (pintype "passive"))
+    (pad "3" thru_hole oval (at 0 5.08 90) (size 1.7 1.7) (drill 1) (layers *.Cu *.Mask)
+      (net 151 "/Connectors/TRQ") (pinfunction "Pin_3") (pintype "passive"))
+    (pad "4" thru_hole oval (at 0 7.62 90) (size 1.7 1.7) (drill 1) (layers *.Cu *.Mask)
+      (net 151 "/Connectors/TRQ") (pinfunction "Pin_4") (pintype "passive"))
+    (pad "5" thru_hole oval (at 0 10.16 90) (size 1.7 1.7) (drill 1) (layers *.Cu *.Mask)
+      (net 152 "/Connectors/GND") (pinfunction "Pin_5") (pintype "passive"))
+    (pad "6" thru_hole oval (at 0 12.7 90) (size 1.7 1.7) (drill 1) (layers *.Cu *.Mask)
+      (net 152 "/Connectors/GND") (pinfunction "Pin_6") (pintype "passive"))
+    (pad "7" thru_hole oval (at 0 15.24 90) (size 1.7 1.7) (drill 1) (layers *.Cu *.Mask)
+      (net 153 "/Connectors/VREF") (pinfunction "Pin_7") (pintype "passive"))
+    (pad "8" thru_hole oval (at 0 17.78 90) (size 1.7 1.7) (drill 1) (layers *.Cu *.Mask)
+      (net 153 "/Connectors/VREF") (pinfunction "Pin_8") (pintype "passive"))
+    (model "${KICAD6_3DMODEL_DIR}/Connector_PinHeader_2.54mm.3dshapes/PinHeader_1x08_P2.54mm_Vertical.wrl"
+      (offset (xyz 0 0 0))
+      (scale (xyz 1 1 1))
