File: Hardware/Testbench_stepper/testbench_stepper.kicad_sch (KiCad schematic)
At the start: 7 parts, among them J1 Conn_01x08_Male, U1 LM358P

Commit message: hw: schematic update
Parts:
- removed C1: 0.1u, symbol Device:C
- removed C2: 100n, symbol Device:C
- removed J1: Conn_01x08_Male, symbol Connector:Conn_01x08_Male
- removed R1: 10k, symbol Device:R
- removed R2: 2K, symbol Device:R
- removed R3: 33K, symbol Device:R
- removed U1: LM358P, symbol EncoderLib:LM358P
Other:
- added sheet Power (power.kicad_sch)
- sheet Connectors ports: added TRQ, VDD_TORQUE, V_SUPPLY+; removed none
- sheet Sensing ports: added TRQ, VDD_TORQUE, V_SUPPLY; removed none
- note removed: "BLACK"
- note removed: "BROWN"
- note removed: "GREY"
- note removed: "WHITE"
