File: Hardware/kicad-project/_autosave-sensing.kicad_sch (KiCad schematic)
At the start: 34 parts, among them U1 LM358P, U2 LEM-CAS-6NP, U3 LM358P, U4 LM358P

Commit message: hw: schematic update
Parts:
- gave numbers to parts that had none: 12
Changed lines of the file:
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@@
   (symbol (lib_id "Device:R") (at 142.875 137.16 0) (unit 1)
     (in_bom yes) (on_board yes) (fields_autoplaced)
-    (property "Reference" "R?" (id 0) (at 144.78 135.8899 0)
+    (property "Reference" "R23" (id 0) (at 144.78 135.8899 0)
       (effects (font (size 1.27 1.27)) (justify left))
     )
@@
   (symbol (lib_id "Device:C") (at 58.42 142.875 270) (unit 1)
     (in_bom yes) (on_board yes) (fields_autoplaced)
-    (property "Reference" "C?" (id 0) (at 58.42 135.255 90))
+    (property "Reference" "C17" (id 0) (at 58.42 135.255 90))
     (property "Value" "C" (id 1) (at 58.42 137.795 90))
     (property "Footprint" "Capacitor_SMD:C_0805_2012Metric" (id 2) (at 54.61 143.8402 0)
@@
   (symbol (lib_id "Device:R") (at 20.32 124.46 270) (unit 1)
     (in_bom yes) (on_board yes)
-    (property "Reference" "R?" (id 0) (at 20.32 122.555 90))
+    (property "Reference" "R15" (id 0) (at 20.32 122.555 90))
     (property "Value" "0" (id 1) (at 20.32 124.46 90))
     (property "Footprint" "Resistor_SMD:R_0603_1608Metric" (id 2) (at 20.32 122.682 90)
@@
   (symbol (lib_id "Device:C") (at 243.84 122.555 270) (unit 1)
     (in_bom yes) (on_board yes) (fields_autoplaced)
-    (property "Reference" "C?" (id 0) (at 243.84 114.935 90))
+    (property "Reference" "C19" (id 0) (at 243.84 114.935 90))
     (property "Value" "C" (id 1) (at 243.84 117.475 90))
     (property "Footprint" "Capacitor_SMD:C_0805_2012Metric" (id 2) (at 240.03 123.5202 0)
@@
   (symbol (lib_id "Device:R") (at 125.73 54.61 0) (unit 1)
     (in_bom yes) (on_board yes)
-    (property "Reference" "R?" (id 0) (at 123.825 54.61 90))
+    (property "Reference" "R22" (id 0) (at 123.825 54.61 90))
     (property "Value" "0" (id 1) (at 125.73 54.61 90))
     (property "Footprint" "Resistor_SMD:R_0603_1608Metric" (id 2) (at 123.952 54.61 90)
@@
   (symbol (lib_id "Device:R") (at 50.8 153.035 0) (unit 1)
     (in_bom yes) (on_board yes) (fields_autoplaced)
-    (property "Reference" "R?" (id 0) (at 52.705 151.7649 0)
+    (property "Reference" "R16" (id 0) (at 52.705 151.7649 0)
       (effects (font (size 1.27 1.27)) (justify left))
     )
@@
   (symbol (lib_id "Device:R") (at 207.645 54.61 0) (unit 1)
     (in_bom yes) (on_board yes)
-    (property "Reference" "R?" (id 0) (at 209.55 53.3399 0)
+    (property "Reference" "R25" (id 0) (at 209.55 53.3399 0)
       (effects (font (size 1.27 1.27)) (justify left))
     )
@@
   (symbol (lib_id "power:GND") (at 142.875 140.97 0) (unit 1)
     (in_bom yes) (on_board yes) (fields_autoplaced)
-    (property "Reference" "#PWR?" (id 0) (at 142.875 147.32 0)
+    (property "Reference" "#PWR0137" (id 0) (at 142.875 147.32 0)
       (effects (font (size 1.27 1.27)) hide)
     )
@@
   (symbol (lib_id "power:GND") (at 50.8 156.845 0) (unit 1)
     (in_bom yes) (on_board yes) (fields_autoplaced)
-    (property "Reference" "#PWR?" (id 0) (at 50.8 163.195 0)
+    (property "Reference" "#PWR0135" (id 0) (at 50.8 163.195 0)
       (effects (font (size 1.27 1.27)) hide)
     )
@@
   (symbol (lib_id "Device:R") (at 150.495 133.35 90) (unit 1)
     (in_bom yes) (on_board yes)
-    (property "Reference" "R?" (id 0) (at 150.495 136.525 90))
+    (property "Reference" "R24" (id 0) (at 150.495 136.525 90))
     (property "Value" "R" (id 1) (at 150.495 130.81 90))
     (property "Footprint" "Resistor_SMD:R_0603_1608Metric" (id 2) (at 150.495 135.128 90)
@@
   (symbol (lib_id "Device:C") (at 150.495 127 270) (unit 1)
     (in_bom yes) (on_board yes) (fields_autoplaced)
-    (property "Reference" "C?" (id 0) (at 150.495 119.38 90))
+    (property "Reference" "C18" (id 0) (at 150.495 119.38 90))
     (property "Value" "C" (id 1) (at 150.495 121.92 90))
     (property "Footprint" "Capacitor_SMD:C_0805_2012Metric" (id 2) (at 146.685 127.9652 0)
@@
   (symbol (lib_id "Device:R") (at 236.22 132.715 0) (unit 1)
     (in_bom yes) (on_board yes) (fields_autoplaced)
-    (property "Reference" "R?" (id 0) (at 238.125 131.4449 0)
+    (property "Reference" "R26" (id 0) (at 238.125 131.4449 0)
       (effects (font (size 1.27 1.27)) (justify left))
     )
@@
   (symbol (lib_id "Device:R") (at 58.42 149.225 90) (unit 1)
     (in_bom yes) (on_board yes)
-    (property "Reference" "R?" (id 0) (at 58.42 152.4 90))
+    (property "Reference" "R17" (id 0) (at 58.42 152.4 90))
     (property "Value" "R" (id 1) (at 58.42 146.685 90))
     (property "Footprint" "Resistor_SMD:R_0603_1608Metric" (id 2) (at 58.42 151.003 90)
@@
   (symbol (lib_id "power:GND") (at 236.22 136.525 0) (unit 1)
     (in_bom yes) (on_board yes) (fields_autoplaced)
-    (property "Reference" "#PWR?" (id 0) (at 236.22 142.875 0)
+    (property "Reference" "#PWR0138" (id 0) (at 236.22 142.875 0)
       (effects (font (size 1.27 1.27)) hide)
     )
@@
   (symbol (lib_id "Device:R") (at 243.84 128.905 90) (unit 1)
     (in_bom yes) (on_board yes)
-    (property "Reference" "R?" (id 0) (at 243.84 132.08 90))
+    (property "Reference" "R27" (id 0) (at 243.84 132.08 90))
     (property "Value" "R" (id 1) (at 243.84 126.365 90))
     (property "Footprint" "Resistor_SMD:R_0603_1608Metric" (id 2) (at 243.84 130.683 90)
