File: Hardware/kicad-project/_autosave-connectors.kicad_sch (KiCad schematic)
At the start: 25 parts, among them CN10 Conn_02x17_Odd_Even, CN7 Conn_02x10_Odd_Even, CN8 Conn_02x08_Odd_Even, CN9 Conn_02x15_Odd_Even, J1 Brake connector, J2 Conn_01x08, J3 PWM module connector, J5 UART Connector, J6 Stepper supply, Q1 Q_NMOS_DGS

Commit message: hw: first pcb routing
Parts:
- renumbered TP_12V to TP_12V1, TP_24V to TP_24V1, TP_5V to TP_5V1, TP_BRAKE to TP_BRAKE1, TP_TORQUE to TP_TORQUE1
Changed lines of the file:
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@@
   (symbol (lib_id "Connector:TestPoint") (at 47.625 152.4 180) (unit 1)
     (in_bom yes) (on_board yes) (fields_autoplaced)
-    (property "Reference" "TP_12V" (id 0) (at 49.53 154.4319 0)
+    (property "Reference" "TP_12V1" (id 0) (at 49.53 154.4319 0)
       (effects (font (size 1.27 1.27)) (justify right))
     )
@@
   (symbol (lib_id "Connector:TestPoint") (at 62.865 152.4 180) (unit 1)
     (in_bom yes) (on_board yes) (fields_autoplaced)
-    (property "Reference" "TP_5V" (id 0) (at 64.77 154.4319 0)
+    (property "Reference" "TP_5V1" (id 0) (at 64.77 154.4319 0)
       (effects (font (size 1.27 1.27)) (justify right))
     )
@@
   (symbol (lib_id "Connector:TestPoint") (at 33.655 152.4 180) (unit 1)
     (in_bom yes) (on_board yes) (fields_autoplaced)
-    (property "Reference" "TP_24V" (id 0) (at 35.56 154.4319 0)
+    (property "Reference" "TP_24V1" (id 0) (at 35.56 154.4319 0)
       (effects (font (size 1.27 1.27)) (justify right))
     )
@@
   (symbol (lib_id "Connector:TestPoint") (at 40.64 170.18 180) (unit 1)
     (in_bom yes) (on_board yes) (fields_autoplaced)
-    (property "Reference" "TP_TORQUE" (id 0) (at 43.18 172.2119 0)
+    (property "Reference" "TP_TORQUE1" (id 0) (at 43.18 172.2119 0)
       (effects (font (size 1.27 1.27)) (justify right))
     )
@@
   (symbol (lib_id "Connector:TestPoint") (at 63.5 170.815 180) (unit 1)
     (in_bom yes) (on_board yes) (fields_autoplaced)
-    (property "Reference" "TP_BRAKE" (id 0) (at 65.405 172.8469 0)
-      (effects (font (size 1.27 1.27)) (justify right))
-    )
+    (property "Reference" "TP_BRAKE1" (id 0) (at 65.405 172.8469 0)
+      (effects (font (size 1.27 1.27)) (justify right))
+    )
