File: Hardware/kicad-project/_autosave-stepper_testbench.kicad_pcb (KiCad board)
At the start: 2 copper layers, 67.7 x 76.7 mm, 77 parts, among them CN10 Conn_02x17_Odd_Even, CN7 Conn_02x10_Odd_Even, CN8 Conn_02x08_Odd_Even, CN9 Conn_02x15_Odd_Even, J1 Brake connector, J2 Conn_01x08, J3 PWM module connector, J4 Conn_01x02, J5 UART Connector, J6 Stepper supply, Q1 Q_NMOS_DGS, U1 LM358P, U2 LEM-CAS-6NP, U3 LM358P, U4 LM358P, U5 LM7812_TO220, U6 L7805

Commit message: hw: update layout corrections
Parts:
- moved TP2 17.5 mm to (142.2, 130.3)
- moved TP1 2.55 mm to (127.0, 71.1)
- moved J6 2.30 mm to (120.1, 69.3)
Routing:
- net /Connectors/TORQUE: track 37.4 -> 25.5 mm
- net GND: vias 96 -> 99
Other:
- board text added: "+12V"
- board text added: "+5V"
- board text added: "TORQUE"
- board text added: "TORQUE TRANSDUCER"
- board text removed: "TORQUE TRANSDUCER CONNECTOR"
