File: Hardware/kicad-project/_autosave-stepper_testbench.kicad_pcb (KiCad board)
At the start: 2 copper layers, 67.7 x 78.4 mm, 76 parts, among them CN10 Conn_02x17_Odd_Even, CN7 Conn_02x10_Odd_Even, CN8 Conn_02x08_Odd_Even, CN9 Conn_02x15_Odd_Even, J1 Brake connector, J2 Conn_01x08, J4 Conn_01x02, J5 UART Connector, J6 Stepper supply, Q1 Q_NMOS_DGS, Q2 Q_NMOS_DGS, U1 LM358P, U2 LEM-CAS-6NP, U3 LM358P, U4 LM358P, U5 LM7812_TO220, U6 L7805

Commit message: hw: final pdf schematic upload
Connections:
- CN7 pad 12: /Connectors/PWM_BRAKE -> unconnected-(CN7-Pad12)
- CN8 pad 2: unconnected-(CN8-Pad2) -> /Connectors/PWM_BRAKE
- CN8 pad 4: unconnected-(CN8-Pad4) -> /Connectors/DISABLE_STEPPER_SUPPLY
