File: Hardware/kicad-project/power.kicad_sch (KiCad schematic)
At the start: 18 parts, among them J4 Conn_01x02, U5 LM317_TO-263, U6 L7805

Commit message: hw: schematic update
Parts:
- removed C9: 1u, symbol Device:C
- removed D5: 1N4002, Diode_SMD:D_SOD-323, symbol Diode:1N4002
- removed R15: 4k7, Resistor_SMD:R_0603_1608Metric, symbol Device:R
- removed R16: 3k9, Resistor_SMD:R_0603_1608Metric, symbol Device:R
- removed R17: 1k, Resistor_SMD:R_0603_1608Metric, symbol Device:R
- removed U5: LM317_TO-263, Package_TO_SOT_THT:TO-220-3_Vertical, symbol Regulator_Linear:LM317_TO-263
- added C12: 0.1u, Capacitor_SMD:C_0603_1608Metric, symbol Device:C
- added C13, C15: 0.33u_DNP, Capacitor_THT:CP_Radial_D5.0mm_P2.50mm, symbol Device:C
- added C14, C16: 0.1u_DNP, Capacitor_THT:CP_Radial_D5.0mm_P2.50mm, symbol Device:C
- added U5: LM7812_TO220, Package_TO_SOT_THT:TO-220-3_Vertical, symbol Regulator_Linear:LM7812_TO220
- C10: footprint (none) -> Capacitor_SMD:C_0603_1608Metric; V (none) -> 25V
- C11: footprint (none) -> Capacitor_SMD:C_0603_1608Metric
- C8: value 0.1u -> 0.33u; footprint (none) -> Capacitor_SMD:C_0603_1608Metric; V (none) -> 25V
- D2, D3: footprint (none) -> Diode_SMD:D_SOD-323
- gave numbers to parts that had none: 2
Connections:
- net +12V: now also C12.1, C14.1, C15.1, U5.3 (VO)
- net +24V: now also C13.1, U5.1 (VI)
- net +5V: now also C16.1
- net GND: now also C12.2, C13.2, C14.2, C15.2, C16.2, U5.2 (GND)
Other:
- moved on the sheet: C10, C11, D2, D3, D4, D6, FB1, J4, R20, R21, U6

Commit message: change 24V zener footprint to SMA
Parts:
- D2: footprint Diode_SMD:D_SOD-323 -> Diode_SMD:D_SMA
Changed lines of the file:
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@@
     (property "Reference" "D2" (id 0) (at 87.63 87.63 0))
     (property "Value" "DIODE" (id 1) (at 87.63 90.17 0))
-    (property "Footprint" "Diode_SMD:D_SOD-323" (id 2) (at 87.63 93.98 0)
+    (property "Footprint" "Diode_SMD:D_SMA" (id 2) (at 87.63 93.98 0)
       (effects (font (size 1.27 1.27)) hide)
     )

Commit message: hw: sch update
Parts:
- D2: footprint Diode_SMD:D_SMA -> Diode_SMD:D_SOD-323
- D3: footprint Diode_SMD:D_SOD-323 -> Diode_SMD:D_SMA
Changed lines of the file:
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@@
     (property "Reference" "D2" (id 0) (at 87.63 87.63 0))
     (property "Value" "DIODE" (id 1) (at 87.63 90.17 0))
-    (property "Footprint" "Diode_SMD:D_SMA" (id 2) (at 87.63 93.98 0)
+    (property "Footprint" "Diode_SMD:D_SOD-323" (id 2) (at 87.63 93.98 0)
       (effects (font (size 1.27 1.27)) hide)
     )
@@
       (effects (font (size 1.27 1.27)) (justify left))
     )
-    (property "Footprint" "Diode_SMD:D_SOD-323" (id 2) (at 93.98 98.425 0)
-      (effects (font (size 1.27 1.27)) hide)
-    )
+    (property "Footprint" "Diode_SMD:D_SMA" (id 2) (at 93.98 98.425 0)
+      (effects (font (size 1.27 1.27)) hide)
+    )

Commit message: hw: final pdf schematic upload
Connections:
- net VIN: now reaches FB1.1, J4.2 (Pin_2)
Other:
- note added: "POWER MANAGEMENT"
- note removed: "V_SUPPLY"
- moved on the sheet: C10, C11, C12, C13, C14, C15, C16, C8, D2, D3, D4, D6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
