File: Hardware/kicad-project/stepper_testbench.kicad_sch (KiCad schematic)
At the start: 0 parts

Commit message: hw: layout v0.1.1
Other:
- sheet Connectors ports: added STEPPER+; removed CURRENT_IN, CURRENT_OUT
- sheet Sensing ports: added STEPPER+; removed COIL_IN, COIL_OUT
Changed lines of the file:
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@@
 (kicad_sch (version 20211123) (generator eeschema)
   (paper "A4")
-  (wire (pts (xy 111.76 83.82) (xy 142.24 83.82))
+  (wire (pts (xy 111.76 85.852) (xy 142.24 85.852))
     (stroke (width 0) (type default) (color 0 0 0 0))
   )
@@
   )
   (wire (pts (xy 111.76 78.74) (xy 142.24 78.74))
-    (stroke (width 0) (type default) (color 0 0 0 0))
-  )
-  (wire (pts (xy 111.76 85.725) (xy 142.24 85.725))
     (stroke (width 0) (type default) (color 0 0 0 0))
   )
@@
       (effects (font (size 1.27 1.27)) (justify right))
     )
-    (pin "CURRENT_IN" input (at 111.76 83.82 0)
-      (effects (font (size 1.27 1.27)) (justify right))
-    )
-    (pin "CURRENT_OUT" input (at 111.76 85.725 0)
-      (effects (font (size 1.27 1.27)) (justify right))
-    )
     (pin "CURRENT_ADC" input (at 111.76 92.71 0)
       (effects (font (size 1.27 1.27)) (justify right))
@@
     )
     (pin "VOLTAGE_STEPPER_ADC" input (at 111.76 97.79 0)
+      (effects (font (size 1.27 1.27)) (justify right))
+    )
+    (pin "STEPPER+" input (at 111.76 85.852 0)
       (effects (font (size 1.27 1.27)) (justify right))
     )
@@
       (effects (font (size 1.27 1.27)) (justify left))
     )
-    (pin "COIL_IN" input (at 142.24 83.82 180)
-      (effects (font (size 1.27 1.27)) (justify left))
-    )
     (pin "CURRENT_BUFF_ADC" input (at 142.24 92.71 180)
-      (effects (font (size 1.27 1.27)) (justify left))
-    )
-    (pin "COIL_OUT" input (at 142.24 85.725 180)
       (effects (font (size 1.27 1.27)) (justify left))
     )
@@
       (effects (font (size 1.27 1.27)) (justify left))
     )
+    (pin "STEPPER+" input (at 142.24 85.852 180)
+      (effects (font (size 1.27 1.27)) (justify left))
+    )
