File: Hardware/kicad-project/stepper_testbench.kicad_pcb (KiCad board)
At the start: 2 copper layers, 67.7 x 78.4 mm, 76 parts, among them CN10 Conn_02x17_Odd_Even, CN7 Conn_02x10_Odd_Even, CN8 Conn_02x08_Odd_Even, CN9 Conn_02x15_Odd_Even, J1 Brake connector, J2 Conn_01x08, J4 Conn_01x02, J5 UART Connector, J6 Stepper supply, Q1 Q_NMOS_DGS, Q2 Q_NMOS_DGS, U1 LM358P, U2 LEM-CAS-6NP, U3 LM358P, U4 LM358P, U5 LM7812_TO220, U6 L7805

Commit message: hw: layout v0.1.1
Parts:
- moved TP5 25.8 mm to (150.1, 62.5)
- moved R27 11.8 mm to (141.5, 105.3), turned to 0 degrees
- moved U2 9.60 mm to (148.6, 80.7), turned to -90 degrees
- moved C2 8.74 mm to (151.9, 72.9), turned to 180 degrees
- moved C9 7.49 mm to (145.5, 73.9), turned to 0 degrees
- moved R2 7.29 mm to (145.6, 72.0), turned to 180 degrees
- moved R23 7.09 mm to (161.1, 106.4), turned to 0 degrees
- moved R16 6.77 mm to (161.1, 91.6), turned to 0 degrees
- moved R17 6.44 mm to (161.1, 85.0), turned to 0 degrees
- moved R24 6.12 mm to (161.1, 99.8), turned to 0 degrees
- moved J6 5.08 mm to (137.4, 50.0), turned to 0 degrees
- moved C19 4.97 mm to (141.5, 101.9), turned to 180 degrees
- moved C6 4.06 mm to (155.8, 104.1)
- moved R12 4.06 mm to (157.5, 104.1)
- moved R14 4.06 mm to (155.8, 97.5)
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Connections:
- CN7 pad 12: /Connectors/PWM_BRAKE -> unconnected-(CN7-Pad12)
- CN8 pad 2: unconnected-(CN8-Pad2) -> /Connectors/PWM_BRAKE
- CN8 pad 4: unconnected-(CN8-Pad4) -> /Connectors/ENABLE_STEPPER_SUPPLY
- R5 pad 1: /Connectors/DISABLE_STEPPER_SUPPLY -> /Connectors/ENABLE_STEPPER_SUPPLY
- U2 pad 7: /Sensing/STEPPER+ -> /Connectors/STEPPER+
- U2 pad 8: /Sensing/STEPPER+ -> /Connectors/STEPPER+
- U2 pad 9: /Sensing/STEPPER+ -> /Connectors/STEPPER+
Routing:
- net +24V: track 0.00 -> 102.6 mm, vias 0 -> 2
- net +12V: track 0.00 -> 75.3 mm, vias 0 -> 2
- net +5V: track 0.00 -> 73.5 mm, vias 0 -> 1
- net /Sensing/CURRENT_BUFF_ADC: track 0.00 -> 46.6 mm, vias 0 -> 1
- net /Sensing/TORQUE_BUFF_ADC: track 0.00 -> 44.3 mm
- net /Sensing/CURRENT_SENSOR_OUTPUT: track 0.00 -> 43.2 mm, vias 0 -> 3
- net /Connectors/TORQUE: track 0.00 -> 35.3 mm, vias 0 -> 2
- net /Connectors/STEPPER+: track 0.00 -> 34.3 mm
- net /Sensing/VOLTAGE_STEPPER_BUFF_ADC: track 0.00 -> 29.1 mm
- net /Connectors/PWM_BRAKE: track 0.00 -> 20.9 mm, vias 0 -> 1
- net Net-(Q2-Pad2): track 0.00 -> 16.7 mm, vias 0 -> 9
- net /Sensing/TORQUE_BUFF: track 0.00 -> 15.1 mm
- net /Sensing/CURRENT_BUFF: track 0.00 -> 15.0 mm
- net /Sensing/V_SUPPLY_BUFF: track 0.00 -> 14.6 mm
- net /Sensing/ADC_V_SUPPLY: track 0.00 -> 13.5 mm
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Other:
- board text added: "+"
- board text added: "-"
- board text added: "PWM BRAKE"
- board text added: "STB - Rev 0.1 Expansion board for NUCLEO-H723ZG"
- board text removed: "+24V"
- board text removed: "+5V"
- board text removed: "STB expansion board for NUCLEO-H723ZG - Rev 0.1"
- board text removed: "led D6 e D4 vicini"
- board text removed: "led o test point entrambi non ha senso"
- board text removed: "nomi led"

Commit message: hw: layout v0.1.2
Routing:
- net GND: vias 91 -> 96
- added copper zone on F.Cu, net Net-(Q1-Pad2)
- added copper zone on F.Cu, net Net-(Q2-Pad2)
